Commit message: Remove DVL integration and related configurations from the simulation

File: packages/bluerov_sim/urdf/bluerov2.urdf (robot description, URDF)
Before this commit: robot bluerov2, 15 links, 14 joints
Links:
- removed link dvl_link
Joints:
- removed joint dvl_joint

Commit message: Add nvidia offload for increase rtf and remove world_objects_to_markers.py

File: packages/bluerov_sim/urdf/bluerov2.urdf (robot description, URDF)
Before this commit: robot bluerov2, 14 links, 13 joints
Joints:
- joint torpedo_shooter_left_joint: origin xyz=0.20 0.05 0.0 rpy=0 0 0 -> xyz=0.20 0.0135 0.0 rpy=0 0 0
- joint torpedo_shooter_right_joint: origin xyz=0.20 -0.05 0.0 rpy=0 0 0 -> xyz=0.20 -0.0135 0.0 rpy=0 0 0

Commit message: Revert torpedo link poses

File: packages/bluerov_sim/urdf/bluerov2.urdf (robot description, URDF)
Before this commit: robot bluerov2, 14 links, 13 joints
Joints:
- joint torpedo_shooter_left_joint: origin xyz=0.20 0.0135 0.0 rpy=0 0 0 -> xyz=0.20 0.05 0.0 rpy=0 0 0
- joint torpedo_shooter_right_joint: origin xyz=0.20 -0.0135 0.0 rpy=0 0 0 -> xyz=0.20 -0.05 0.0 rpy=0 0 0
